Commit message: adding visual stl and modify base

File: myturtle_description/urdf/myturtle_base.urdf.xacro (robot description, xacro)
@@ -20,6 +20,8 @@
     <visual>
       <geometry>
-        <cylinder length="${base_collision_height}" radius="${base_collision_radius}"/>
-      </geometry>
+        <!-- <cylinder length="${base_collision_height}" radius="${base_collision_radius}"/> -->
+        <mesh filename="package://myturtle_description/mesh/myturtle_visual.STL"/>
+      </geometry>
+      <origin xyz="0 0 -${base_collision_height/2}" rpy="${M_PI/2} 0 ${M_PI/2}"/>
       <material name="white">
         <color rgba="1 1 1 1"/>
@@ -79,5 +81,5 @@
     <parent link="base_link"/>
     <child link="left_wheel_link"/>
-    <origin xyz="0 ${wheels_distance/2} ${wheel_center_offset-base_collision_height/2}" rpy="${M_PI/2} 0 0"/>
+    <origin xyz="0 ${wheels_distance/2} ${wheel_center_offset-base_collision_height/2}" rpy="${-M_PI/2} 0 0"/>
     <axis xyz="0 0 1"/>
   </joint>
@@ -109,5 +111,5 @@
     <parent link="base_link"/>
     <child link="right_wheel_link"/>
-    <origin xyz="0 -${wheels_distance/2} ${wheel_center_offset-base_collision_height/2}" rpy="${M_PI/2} 0 0"/>
+    <origin xyz="0 -${wheels_distance/2} ${wheel_center_offset-base_collision_height/2}" rpy="${-M_PI/2} 0 0"/>
     <axis xyz="0 0 1"/>
   </joint>
